Commit message: add camera simulation and fix main processor

File: src/whitepost_description/urdf/whitepost_description.urdf (robot description, URDF)
Before this commit: robot whitepost_description, 6 links, 5 joints
Links:
- link link5: mass 0.0824040605350861 -> 0.0824040607022898
Joints:
- joint joint1: origin xyz=-0.015946 -0.24025 0.058318 rpy=0 0 0 -> xyz=-0.0159462258519159 -0.240246042857508 0.0583181110479435 rpy=0 0 0
- joint joint2: origin xyz=0.073496 -0.005504 0.045 rpy=-1.5708 0 1.5708 -> xyz=0.0734962258519162 -0.00550395714249205 0.0449999999999996 rpy=-1.5707963267949 0 1.5707963267949
- joint joint3: origin xyz=-0.56889 5E-05 0.068996 rpy=0 0 0 -> xyz=-0.568892521556106 5.00000000043382E-05 0.0689962258519109 rpy=0 0 0
- joint joint5: origin xyz=0.0296 -0.0748 -0.0408 rpy=3.1416 1.5708 0 -> xyz=-0.0295999999999965 -0.0748000000000026 -0.0408000000000002 rpy=0 -1.5707963267949 3.14159265358979
